File: expansion.kicad_sch (KiCad schematic)
At the start: 3 parts, among them J2 UART, J3 EXPANSION, J5 Solder Pads

Commit message: we are no longer an official project of the All Things Linux 501(c)(3) organization
Other:
- title: (none) -> Tux Keychain
Changed lines of the file:
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@@
 	(generator_version "9.0")
 	(paper "A4")
+	(title_block
+		(title "Tux Keychain")
+		(date "2025-05-19")
+		(rev "2")
+	)
 	(text "do not populate by default"
 		(exclude_from_sim no)
