File: tuxkeychain.kicad_sch (KiCad schematic)
At the start: 44 parts, among them J1 Amphenol_10104111, Q2 2N7002, SW1 RESET, SW2 FEL, U4 F1C100s, U5 TLV76701DRVx, U6 W25Q128JVS, U7 TLV76701DRVx, U8 TLV76701DRVx, Y1 24MHz

Commit message: we are no longer an official project of the All Things Linux 501(c)(3) organization
Other:
- company: All Things Linux 501(c)(3)  -> (none)
Changed lines of the file:
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@@
 		(date "2025-05-19")
 		(rev "2")
-		(company "All Things Linux 501(c)(3) ")
 	)
 	(text "red for extra ominous points"
