File: tuxkeychain.kicad_pcb (KiCad board)
At the start: 6 copper layers, 50 x 60 mm, 56 parts, among them J1 Amphenol_10104111, J2 UART, J3 EXPANSION, J5 Solder Pads, Q2 2N7002, SW1 RESET, SW2 FEL, U4 F1C100s, U5 TLV76701DRVx, U6 W25Q128JVS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

Commit message: change text
Other:
- board text added: "electron271.gay"
- board text removed: "allthingslinux.org"
Changed lines of the file:
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@@
 			(size 4 4)
 			(drill 4)
-			(layers "F&B.Cu" "*.Mask")
+			(layers "*.Cu" "*.Mask")
 			(clearance 0.1)
 			(zone_connect 0)
@@
 		(layer "Edge.Cuts")
 	)
-	(gr_text "allthingslinux.org\n"
+	(gr_text "electron271.gay\n"
 		(locked yes)
 		(at 129 108 15)
