File: expansion/expansion.kicad_sch (KiCad schematic)
At the start: 5 parts, among them J1 Micro_SD_Card_Det2, J2 TRRS, J3 EXPANSION, J4 R, J5 L

Commit message: we are no longer an official project of the All Things Linux 501(c)(3) organization
Other:
- company: All Things Linux 501(c)(3) -> (none)
Changed lines of the file:
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@@
 		(date "2025-05-24")
 		(rev "1")
-		(company "All Things Linux 501(c)(3)")
 	)
 	(junction
